Commit message: change mass property for kinova

File: examples/rsc/anymalC_kinova/urdf/anymal_kinova front.urdf (robot description, URDF)
Before this commit: robot anymal, 97 links, 96 joints
Links:
- link base_link: mass 1.697 -> 0.697
- link bicep_link: mass 1.262 -> 0.262
- link bracelet_link: mass 0.5 -> 0.2
- link forearm_link: mass 0.93 -> 0.23
- link robotiq_arg2f_base_link: mass 0.22652 -> 0.02652
- link shoulder_link: mass 1.377 -> 0.377
- link spherical_wrist_1_link: mass 0.6781 -> 0.1781
- link spherical_wrist_2_link: mass 0.678 -> 0.178

Commit message: finger collision param update

File: examples/rsc/anymalC_kinova/urdf/anymal_kinova front.urdf (robot description, URDF)
Before this commit: robot anymal, 97 links, 96 joints
Links:
- link left_inner_finger_pad: geometry collision box size=0.022 0.01035 0.0375; visual box size=0.022 0.00635 0.0375
- link right_inner_finger_pad: geometry collision box size=0.022 0.01035 0.0375; visual box size=0.022 0.00635 0.0375

Commit message: modify the position of kinova base

File: examples/rsc/anymalC_kinova/urdf/anymal_kinova front.urdf (robot description, URDF)
Before this commit: robot anymal, 97 links, 96 joints
Joints:
- joint arm_to_anymal: origin xyz=0.35801 0 0.073 rpy=0 0 0 -> xyz=0.49801 0 0.063 rpy=0 0 0

Commit message: different materials for new demo

File: examples/rsc/anymalC_kinova/urdf/anymal_kinova front.urdf (robot description, URDF)
Before this commit: robot anymal, 97 links, 96 joints
Joints:
- joint arm_to_anymal: origin xyz=0.49801 0 0.063 rpy=0 0 0 -> xyz=0.35801 0 0.073 rpy=0 0 0

File: examples/rsc/anymalC_kinova/urdf/anymal_kinova front_buzz_wire.urdf (robot description, URDF)
Before this commit: robot anymal, 87 links, 86 joints
Joints:
- removed joint end_effector
- added joint bracelet_link_to_end_effector: type fixed, parent bracelet_link, child end_effector_link, origin xyz=0 0 -0.0615250000000001 rpy=3.14159265358979 1.09937075168372E-32 3.14159265358979, axis 0 0 0
- joint face_front_to_wide_angle_camera_front_camera: origin xyz=0.09850 0.0 0.01497 rpy=0 0 0 -> xyz=0.0 0.0 0.01497 rpy=0 0 0
