Commit message: add some objects for buzz wire demo

File: examples/rsc/anymalC_kinova/urdf/anymal_kinova front_buzz_wire.urdf (robot description, URDF)
Before this commit: robot anymal, 97 links, 96 joints
Links:
- removed link left_inner_finger
- removed link left_inner_finger_pad
- removed link left_inner_knuckle
- removed link left_outer_finger
- removed link left_outer_knuckle
- removed link right_inner_finger
- removed link right_inner_finger_pad
- removed link right_inner_knuckle
- removed link right_outer_finger
- removed link right_outer_knuckle
- removed link robotiq_arg2f_base_link
- added link donut, mass 1E-06; collision mesh filename=../customize_materials/donut_tip.obj scale=0.0005 0.0005 0.0005; visual mesh filename=../customize_materials/donut_tip.obj scale=0.0005 0.0005 0.0005
- added link tip_stick, mass 1E-06; collision cylinder length=0.09 radius=0.005; visual cylinder length=0.09 radius=0.005
Joints:
- removed joint finger_joint
- removed joint left_inner_finger_joint
- removed joint left_inner_finger_pad_joint
- removed joint left_inner_knuckle_joint
- removed joint left_outer_finger_joint
- removed joint right_inner_finger_joint
- removed joint right_inner_finger_pad_joint
- removed joint right_inner_knuckle_joint
- removed joint right_outer_finger_joint
- removed joint right_outer_knuckle_joint
- added joint tipStick_donut: type fixed, parent tip_stick, child donut, origin xyz=0.0 0.0 0.047 rpy=0.0 0.0 0
- joint gripper_base_joint: child robotiq_arg2f_base_link -> tip_stick; origin xyz=0.0 0.0 0.0 rpy=0.0 0.0 1.57 -> xyz=0.0 0.0 0.0 rpy=0.0 0.0 0

Commit message: change the origin of donut

File: examples/rsc/anymalC_kinova/urdf/anymal_kinova front_buzz_wire.urdf (robot description, URDF)
Before this commit: robot anymal, 88 links, 87 joints
Links:
- removed link tip_stick
- link donut: geometry collision mesh filename=../customize_materials/donut_tip.obj scale=0.0009 0.0009 0.0009; visual mesh filename=../customize_materials/donut_tip.obj scale=0.0009 0.0009 0.0009
Joints:
- removed joint tipStick_donut
- joint gripper_base_joint: child tip_stick -> donut

Commit message: New buzz wire and donut

File: examples/rsc/anymalC_kinova/urdf/anymal_kinova front_buzz_wire.urdf (robot description, URDF)
Before this commit: robot anymal, 87 links, 86 joints
Links:
- removed link donut
- added link end_effector, mass 1E-06; collision mesh filename=../customize_materials/donut_tip.obj scale=0.0005 0.0005 0.0005; visual mesh filename=../customize_materials/donut_tip.obj scale=0.0005 0.0005 0.0005
Joints:
- joint gripper_base_joint: child donut -> end_effector; origin xyz=0.0 0.0 0.0 rpy=0.0 0.0 0 -> xyz=0.0 0.0 0.05 rpy=0.0 0.0 0

Commit message: tiny change of the EE joint for the sake of contact detection

File: examples/rsc/anymalC_kinova/urdf/anymal_kinova front_buzz_wire.urdf (robot description, URDF)
Before this commit: robot anymal, 87 links, 86 joints
Joints:
- joint gripper_base_joint: axis (none) -> 0 0 1; limit (none) -> lower=0 upper=0 effort=0 velocity=0; type fixed -> revolute
